Commit message: Start Chapter6.
Signed-off-by: fgs <ifreewolf@163.com>

File: Chapter6/demo07_ws/src/urdf01_rviz/urdf/urdf/demo04_base_footprint.urdf (robot description, URDF)
Before this commit: robot my_car, 2 links, 1 joints
Links:
- added link base_footprint; visual box size=0.001 0.001 0.001
Joints:
- added joint base_link2base_footprint: type fixed, parent base_footprint, child base_link, origin xyz=0 0 0.05 rpy=0 0 0
