Commit message: Finished arbotix.
Signed-off-by: ifreewolf <ifreewolf@163.com>

File: Chapter6/demo07_ws/src/urdf01_rviz/urdf/xacro/demo06_car_camera.urdf.xacro (robot description, xacro)
@@ -7,10 +7,26 @@
             关节属性：x y z
      -->
-    <xacro:property name="" value="" /> <!--  -->
-    <xacro:property name="" value="" /> <!--  -->
-    <xacro:property name="" value="" /> <!--  -->
-    <xacro:property name="" value="" /> <!--  -->
-    <xacro:property name="" value="" /> <!--  -->
-    <xacro:property name="" value="" /> <!--  -->
+    <xacro:property name="camera_length" value="0.02" /> <!-- 厚度(x) -->
+    <xacro:property name="camera_width" value="0.05" /> <!-- 厚度(y) -->
+    <xacro:property name="camera_height" value="0.05" /> <!-- 高度(z) -->
+    <xacro:property name="joint_camera_x" value="0.08" /> <!--  -->
+    <xacro:property name="joint_camera_y" value="0" /> <!--  -->
+    <xacro:property name="joint_camera_z" value="${base_length / 2 + camera_height / 2}" /> <!--  -->
     <!-- 2.设计连杆和关节 -->
+    <link name="camera">
+        <visual>
+            <origin xyz="0 0 0" rpy="0 0 0" />
+            <geometry>
+                <box size="${camera_length} ${camera_width} ${camera_height}" />
+            </geometry>
+            <matrial name="black">
+                <color rgba="0 0 0 0.8" />
+            </matrial>
+        </visual>
+    </link>
+    <joint name="camera2base" type="fixed">
+        <parent link="base_link" />
+        <child link="camera" />
+        <origin xyz="${joint_camera_x} ${joint_camera_y} ${joint_camera_z}" rpy="0 0 0" />
+    </joint>
 </robot>

File: Chapter6/demo07_ws/src/urdf01_rviz/urdf/xacro/demo07_car_laser.urdf.xacro (robot description, xacro)
@@ -1,3 +1,56 @@
 <robot name="mycar" xmlns:xacro="http://www.ros.org/wiki/xacro">
     <!-- 雷达部件 -->
+    <!-- 参数 -->
+    <!--
+        1.支架
+            支架尺寸：半径 高度
+            关节偏移量：x y z
+        2.雷达
+            雷达尺寸：半径 高度
+            关节偏移量：x y z
+     -->
+    <xacro:property name="support_radius"  value="0.01" />
+    <xacro:property name="support_length"  value="0.15" />
+    <xacro:property name="laser_radius"  value="0.03" />
+    <xacro:property name="laser_length"  value="0.05" />
+    <xacro:property name="joint_support_x"  value="0" />
+    <xacro:property name="joint_support_y"  value="0" />
+    <!-- z = 车体高度 / 2 + 支架高度 / 2 -->
+    <xacro:property name="joint_support_z"  value="${base_length / 2 + support_length / 2}" />
+    <xacro:property name="joint_laser_x"  value="0" />
+    <xacro:property name="joint_laser_y"  value="0" />
+    <!-- z = 支架高度 / 2 + 雷达高度 / 2 -->
+    <xacro:property name="joint_laser_z"  value="${support_length / 2 + laser_length / 2}" />
+    <!-- 1.支架 -->
+    <link name="support">
+        <visual>
+            <geometry>
+                <cylinder radius="${support_radius}" length="${support_length}" />
+            </geometry>
+            <matrial name="yellow">
+                <color rgba="0.8 0.5 0 0.5" />
+            </matrial>
+        </visual>
+    </link>
+    <joint name="support2base" type="fixed">
+        <parent link="base_link" />
+        <child link="support" />
+        <origin xyz="${joint_support_x} ${joint_support_y} ${joint_support_z}" rpy="0 0 0" />
+    </joint>
+    <!-- 2.雷达 -->
+    <link name="laser">
+        <visual>
+            <geometry>
+                <cylinder radius="${laser_radius}" length="${laser_length}" />
+            </geometry>
+            <matrial name="black">
+                <color rgba="0 0 0 0.5" />
+            </matrial>
+        </visual>
+    </link>
+    <joint name="laser2support" type="fixed">
+        <parent link="support" />
+        <child link="laser" />
+        <origin xyz="${joint_laser_x} ${joint_laser_y} ${joint_laser_z}" rpy="0 0 0" />
+    </joint>
 </robot>
